File: stomp_control/stomp_control.kicad_sch (KiCad schematic)
At the start: 0 parts

Commit message: initial schematic design
Connections:
- no-connect marks 0 -> 1
Other:
- added sheet FootSwitches (fs.kicad_sch)
- added sheet MiDi (midi.kicad_sch)
- added sheet PSU (psu.kicad_sch)
- added sheet RP2040 (cpu.kicad_sch)
- added sheet USB (usb.kicad_sch)
