File: stomp_control/midi.kicad_sch (KiCad schematic)
At the start: 3 parts

Commit message: initial board layout
Parts:
- J5: renamed from J?; footprint (none) -> Connector_PinHeader_2.54mm:PinHeader_1x04_P2.54mm_Vertical
- R7, R8: renamed from R?; footprint (none) -> Resistor_SMD:R_0603_1608Metric_Pad0.98x0.95mm_HandSolder
Changed lines of the file:
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@@
   (symbol (lib_id "power:GND") (at 139.7 101.6 0) (unit 1)
     (in_bom yes) (on_board yes)
-    (property "Reference" "#PWR?" (id 0) (at 139.7 107.95 0)
+    (property "Reference" "#PWR0120" (id 0) (at 139.7 107.95 0)
       (effects (font (size 1.27 1.27)) hide)
     )
@@
   (symbol (lib_id "Device:R_Small_US") (at 148.59 85.09 90) (unit 1)
     (in_bom yes) (on_board yes)
-    (property "Reference" "R?" (id 0) (at 144.78 82.55 90))
+    (property "Reference" "R7" (id 0) (at 144.78 82.55 90))
     (property "Value" "33R" (id 1) (at 151.13 82.55 90))
-    (property "Footprint" "" (id 2) (at 148.59 85.09 0)
+    (property "Footprint" "Resistor_SMD:R_0603_1608Metric_Pad0.98x0.95mm_HandSolder" (id 2) (at 148.59 85.09 0)
       (effects (font (size 1.27 1.27)) hide)
     )
@@
   (symbol (lib_id "Device:R_Small_US") (at 148.59 88.9 270) (unit 1)
     (in_bom yes) (on_board yes)
-    (property "Reference" "R?" (id 0) (at 144.78 91.44 90))
+    (property "Reference" "R8" (id 0) (at 144.78 91.44 90))
     (property "Value" "10R" (id 1) (at 151.13 91.44 90))
-    (property "Footprint" "" (id 2) (at 148.59 88.9 0)
+    (property "Footprint" "Resistor_SMD:R_0603_1608Metric_Pad0.98x0.95mm_HandSolder" (id 2) (at 148.59 88.9 0)
       (effects (font (size 1.27 1.27)) hide)
     )
@@
   (symbol (lib_id "Connector:Conn_01x04_Female") (at 125.73 88.9 0) (mirror y) (unit 1)
     (in_bom yes) (on_board yes)
-    (property "Reference" "J?" (id 0) (at 121.92 88.9 0)
+    (property "Reference" "J5" (id 0) (at 121.92 88.9 0)
       (effects (font (size 1.27 1.27)) (justify right))
     )
@@
       (effects (font (size 1.27 1.27)) (justify right))
     )
-    (property "Footprint" "" (id 2) (at 125.73 88.9 0)
+    (property "Footprint" "Connector_PinHeader_2.54mm:PinHeader_1x04_P2.54mm_Vertical" (id 2) (at 125.73 88.9 0)
       (effects (font (size 1.27 1.27)) hide)
     )
