File: stomp_control/psu.kicad_sch (KiCad schematic)
At the start: 11 parts

Commit message: initial board layout
Parts:
- removed U?: LM1117-3.3, symbol Regulator_Linear:LM1117-3.3
- removed U?: LM1117-5.0, symbol Regulator_Linear:LM1117-5.0
- added U3: LM1117MP-5.0_NOPB, Package_TO_SOT_SMD:SOT-223, symbol sc_custom:LM1117MP-5.0_NOPB
- added U4: LMS8117AMP-3.3_NOPB, Package_TO_SOT_SMD:SOT-223, symbol sc_custom:LMS8117AMP-3.3_NOPB
- C10, C11, C12, C7, C8, C9: renamed from C?; footprint (none) -> Capacitor_SMD:C_0603_1608Metric_Pad1.08x0.95mm_HandSolder
- J4: renamed from J?; footprint (none) -> Connector_BarrelJack:BarrelJack_CUI_PJ-102AH_Horizontal
- Q1: renamed from Q?; value Q_PMOS_DGS -> DMG2305UX; footprint (none) -> Package_TO_SOT_SMD:SOT-23
- gave numbers to parts that had none: 1
Connections:
- net 3v3: now also U4.2 (VO), U4.4 (VO)
- net GND: now also U3.1 (GND), U4.1 (GND)
- net at C7.1, J4.2, J4.3: now also U3.3 (VI)
- net at C9.1, D1.1 (K), Q1.3 (S): now also U4.3 (VI)
- net at C8.1, Q1.1 (D): now also U3.2 (VO), U3.4 (VO)
