File: stomp_control/stomp_control.kicad_pcb (KiCad board)
At the start: 0 parts

Commit message: initial board layout
Parts:
- added C1: 15p, Capacitor_SMD:C_0603_1608Metric_Pad1.08x0.95mm_HandSolder, F.Cu at (153.2, 100.0)
- added C10: 10uF, Capacitor_SMD:C_0603_1608Metric_Pad1.08x0.95mm_HandSolder, F.Cu at (148.0, 96.0)
- added C11: 10nF, Capacitor_SMD:C_0603_1608Metric_Pad1.08x0.95mm_HandSolder, F.Cu at (148.0, 98.8)
- added C12: 10nF, Capacitor_SMD:C_0603_1608Metric_Pad1.08x0.95mm_HandSolder, F.Cu at (148.0, 101.8)
- added C13: 100n, Capacitor_SMD:C_0603_1608Metric_Pad1.08x0.95mm_HandSolder, F.Cu at (126.1, 108.2)
- added C14: 100n, Capacitor_SMD:C_0603_1608Metric_Pad1.08x0.95mm_HandSolder, F.Cu at (141.7, 108.1)
- added C15: 100n, Capacitor_SMD:C_0603_1608Metric_Pad1.08x0.95mm_HandSolder, F.Cu at (157.6, 108.1)
- added C16: 100n, Capacitor_SMD:C_0603_1608Metric_Pad1.08x0.95mm_HandSolder, F.Cu at (173.1, 108.1)
- added C2: 15p, Capacitor_SMD:C_0603_1608Metric_Pad1.08x0.95mm_HandSolder, F.Cu at (170.3, 96.0)
- added C3: 100n, Capacitor_SMD:C_0603_1608Metric_Pad1.08x0.95mm_HandSolder, F.Cu at (154.6, 96.0)
- added C4: 100n, Capacitor_SMD:C_0603_1608Metric_Pad1.08x0.95mm_HandSolder, F.Cu at (172.0, 88.0)
- added C5: 2u2, Capacitor_SMD:C_0603_1608Metric_Pad1.08x0.95mm_HandSolder, F.Cu at (172.0, 86.0)
- added C6: 2u2, Capacitor_SMD:C_0603_1608Metric_Pad1.08x0.95mm_HandSolder, F.Cu at (167.1, 81.0)
- added C7: 10uF, Capacitor_SMD:C_0603_1608Metric_Pad1.08x0.95mm_HandSolder, F.Cu at (122.1, 88.9)
- added C8: 10uF, Capacitor_SMD:C_0603_1608Metric_Pad1.08x0.95mm_HandSolder, F.Cu at (136.7, 92.8)
- added C9: 10uF, Capacitor_SMD:C_0603_1608Metric_Pad1.08x0.95mm_HandSolder, F.Cu at (144.1, 81.5)
- added D1: MBR1020VL, Diode_SMD:D_SOD-123F, F.Cu at (136.9, 83.2)
- added H1: MountingHole_Pad, MountingHole:MountingHole_3.2mm_M3_DIN965_Pad, F.Cu at (114.1, 115.5)
- added H2: MountingHole_Pad, MountingHole:MountingHole_3.2mm_M3_DIN965_Pad, F.Cu at (182.6, 115.5)
- added H3: MountingHole_Pad, MountingHole:MountingHole_3.2mm_M3_DIN965_Pad, F.Cu at (114.1, 75.5)
- added H4: MountingHole_Pad, MountingHole:MountingHole_3.2mm_M3_DIN965_Pad, F.Cu at (182.6, 75.5)
- added J1: SWD, Connector_PinHeader_2.54mm:PinHeader_1x03_P2.54mm_Vertical, F.Cu at (178.6, 100.0)
- added J2: PROG_MODE, Connector_PinHeader_2.54mm:PinHeader_1x02_P2.54mm_Vertical, F.Cu at (155.8, 76.0)
- added J3: RESET, Connector_PinHeader_2.54mm:PinHeader_1x02_P2.54mm_Vertical, F.Cu at (178.6, 87.3)
- added J4: 9V center: Neg, Connector_BarrelJack:BarrelJack_CUI_PJ-102AH_Horizontal, F.Cu at (126.4, 82.7)
- added J5: Conn_01x04_Female, Connector_PinHeader_2.54mm:PinHeader_1x04_P2.54mm_Vertical, F.Cu at (173.6, 76.0)
- added J6: FS_1, Connector_PinHeader_2.54mm:PinHeader_1x02_P2.54mm_Vertical, F.Cu at (124.4, 114.0)
- added J7: FS_2, Connector_PinHeader_2.54mm:PinHeader_1x02_P2.54mm_Vertical, F.Cu at (139.9, 114.0)
- added J8: FS_3, Connector_PinHeader_2.54mm:PinHeader_1x02_P2.54mm_Vertical, F.Cu at (155.9, 114.0)
- added J9: FS_4, Connector_PinHeader_2.54mm:PinHeader_1x02_P2.54mm_Vertical, F.Cu at (171.2, 114.0)
- added J?1: USB_C_Receptacle_USB2.0, USB4085-GF-A:GCT_USB4085-GF-A_REVA, F.Cu at (146.6, 73.5)
- added Q1: DMG2305UX, Package_TO_SOT_SMD:SOT-23, F.Cu at (136.9, 88.5)
- added R1: DNF, Resistor_SMD:R_0603_1608Metric_Pad0.98x0.95mm_HandSolder, F.Cu at (160.7, 96.0)
- added R10: 5.1k, Resistor_SMD:R_0603_1608Metric_Pad0.98x0.95mm_HandSolder, F.Cu at (138.1, 76.6)
- added R11: 220k, Resistor_SMD:R_0603_1608Metric_Pad0.98x0.95mm_HandSolder, F.Cu at (123.6, 108.2)
- added R12: 220k, Resistor_SMD:R_0603_1608Metric_Pad0.98x0.95mm_HandSolder, F.Cu at (139.1, 108.1)
- added R13: 220k, Resistor_SMD:R_0603_1608Metric_Pad0.98x0.95mm_HandSolder, F.Cu at (155.1, 108.1)
- added R14: 220k, Resistor_SMD:R_0603_1608Metric_Pad0.98x0.95mm_HandSolder, F.Cu at (170.6, 108.1)
- added R2: 1k, Resistor_SMD:R_0603_1608Metric_Pad0.98x0.95mm_HandSolder, F.Cu at (156.4, 81.0)
- added R3: 1k, Resistor_SMD:R_0603_1608Metric_Pad0.98x0.95mm_HandSolder, F.Cu at (165.8, 96.0)
- added R4: DNF, Resistor_SMD:R_0603_1608Metric_Pad0.98x0.95mm_HandSolder, F.Cu at (153.6, 81.0)
- added R5: 27.4R, Resistor_SMD:R_0603_1608Metric_Pad0.98x0.95mm_HandSolder, B.Cu at (161.2, 80.0)
- added R6: 27.4R, Resistor_SMD:R_0603_1608Metric_Pad0.98x0.95mm_HandSolder, B.Cu at (161.2, 82.0)
- added R7: 33R, Resistor_SMD:R_0603_1608Metric_Pad0.98x0.95mm_HandSolder, F.Cu at (173.1, 81.0)
- added R8: 10R, Resistor_SMD:R_0603_1608Metric_Pad0.98x0.95mm_HandSolder, F.Cu at (170.5, 81.0)
- added R9: 5.1k, Resistor_SMD:R_0603_1608Metric_Pad0.98x0.95mm_HandSolder, F.Cu at (135.6, 76.6)
- added REF**: OSHW-Logo2_24.3x20mm_SilkScreen, Symbol:OSHW-Logo2_24.3x20mm_SilkScreen, F.Cu at (115.5, 99.5)
- added U1: W25Q128JVS, Package_SO:SOIC-8_5.23x5.23mm_P1.27mm, F.Cu at (154.6, 89.0)
- added U2: RP2040, Package_DFN_QFN:QFN-56-1EP_7x7mm_P0.4mm_EP5.6x5.6mm, F.Cu at (164.6, 89.0)
- added U3: LM1117MP-5.0_NOPB, Package_TO_SOT_SMD:SOT-223, F.Cu at (127.9, 91.5)
- added U4: LMS8117AMP-3.3_NOPB, Package_TO_SOT_SMD:SOT-223, F.Cu at (145.4, 89.0)
- added U5: 74HC14, Package_SO:TSSOP-14_4.4x5mm_P0.65mm, F.Cu at (137.6, 99.5)
- added Y1: 12MHz, sc_custom:ABLS-12.000MHZ-20-B-3-H-T, F.Cu at (164.1, 100.0)
Routing:
- net /FootSwitches/3v3: track 0.00 -> 168.1 mm, vias 0 -> 7
- net Net-(C16-Pad1): track 0.00 -> 52.8 mm, vias 0 -> 2
- net /FootSwitches/foot_switch_one: track 0.00 -> 36.5 mm
- net /FootSwitches/foot_switch_two: track 0.00 -> 32.3 mm
- net /FootSwitches/foot_switch_three: track 0.00 -> 32.3 mm
- net /FootSwitches/foot_switch_four: track 0.00 -> 31.4 mm, vias 0 -> 2
- net Net-(C15-Pad1): track 0.00 -> 29.9 mm, vias 0 -> 2
- net Net-(C13-Pad1): track 0.00 -> 26.4 mm, vias 0 -> 2
- net /PSU/VBUS: track 0.00 -> 25.4 mm
- net Net-(C8-Pad1): track 0.00 -> 21.1 mm
- net /RP2040/QSPI_SD0: track 0.00 -> 21.0 mm, vias 0 -> 2
- net Net-(C14-Pad1): track 0.00 -> 20.4 mm, vias 0 -> 2
- net /RP2040/QSPI_CLK: track 0.00 -> 19.9 mm, vias 0 -> 2
- net /USB_-: track 0.00 -> 19.1 mm, vias 0 -> 1
- net /RP2040/~QSPI_CS: track 0.00 -> 18.2 mm
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- added copper zone on B.Cu, net GND
- added copper zone on F.Cu, net GND
Other:
- board outline added: 76.5 x 48 mm
- copper layers 0 -> 2
