File: stomp_control/stomp_control.kicad_pcb (KiCad board)
At the start: 2 copper layers, 76.5 x 48 mm, 53 parts, among them J1 SWD, J2 PROG_MODE, J3 RESET, J4 9V center: Neg, J5 Conn_01x04_Female, J6 FS_1, J7 FS_2, J8 FS_3, J9 FS_4, Q1 DMG2305UX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

Commit message: add silkscreen annotations
Parts:
- renumbered J1 to DEBUG, J?1 to J1
Other:
- board text added: "3v3"
- board text added: "BOOT"
- board text added: "CLK"
- board text added: "Foot Switch 1"
- board text added: "Foot Switch 2"
- board text added: "Foot Switch 3"
- board text added: "Foot Switch 4"
- board text added: "GND"
- board text added: "MiDi"
- board text added: "OUT"
- board text added: "SWD"
- board text added: "~RST"
Changed lines of the file:
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@@
     (pad_to_mask_clearance 0)
     (pcbplotparams
-      (layerselection 0x00010fc_ffffffff)
+      (layerselection 0x00010f0_ffffffff)
       (disableapertmacros false)
       (usegerberextensions false)
@@
       (viasonmask false)
       (mode 1)
-      (useauxorigin false)
+      (useauxorigin true)
       (hpglpennumber 1)
       (hpglpenspeed 20)
@@
       (outputformat 1)
       (mirror false)
-      (drillshape 1)
+      (drillshape 0)
       (scaleselection 1)
-      (outputdirectory "")
+      (outputdirectory "gerbers/")
     )
   )
@@
     (property "Sheetname" "USB")
     (attr through_hole)
-    (fp_text reference "J?1" (at -2.395 -6) (layer "F.SilkS")
+    (fp_text reference "J1" (at -2.395 -6) (layer "F.SilkS")
       (effects (font (size 1.00015 1.00015) (thickness 0.15)))
     )
@@
     (property "Sheetname" "FootSwitches")
     (attr through_hole)
-    (fp_text reference "J9" (at 0 -2.33 90) (layer "F.SilkS")
+    (fp_text reference "J9" (at 0 -2.33 90) (layer "F.SilkS") hide
       (effects (font (size 1 1) (thickness 0.15)))
     )
@@
     (property "Sheetname" "FootSwitches")
     (attr through_hole)
-    (fp_text reference "J6" (at 0 -2.435 270) (layer "F.SilkS")
+    (fp_text reference "J6" (at 0 -2.435 270) (layer "F.SilkS") hide
       (effects (font (size 1 1) (thickness 0.15)))
     )
@@
     (property "Sheetname" "FootSwitches")
     (attr through_hole)
-    (fp_text reference "J7" (at 0 -2.33 90) (layer "F.SilkS")
+    (fp_text reference "J7" (at 0 -2.33 90) (layer "F.SilkS") hide
       (effects (font (size 1 1) (thickness 0.15)))
     )
@@
     (property "Sheetname" "RP2040")
     (attr through_hole)
-    (fp_text reference "J2" (at 0 -2.33 90) (layer "F.SilkS")
+    (fp_text reference "J2" (at 0 -2.33 90) (layer "F.SilkS") hide
       (effects (font (size 1 1) (thickness 0.15)))
     )
@@
     (property "Sheetname" "RP2040")
     (attr through_hole)
-    (fp_text reference "J1" (at 0 -2.33) (layer "F.SilkS")
+    (fp_text reference "DEBUG" (at 0 -2.33) (layer "F.SilkS")
       (effects (font (size 1 1) (thickness 0.15)))
     )
@@
     (property "Sheetname" "MiDi")
     (attr through_hole)
-    (fp_text reference "J5" (at 0 -2.33 90) (layer "F.SilkS")
+    (fp_text reference "J5" (at 0 -2.33 90) (layer "F.SilkS") hide
       (effects (font (size 1 1) (thickness 0.15)))
     )
@@
     (property "Sheetname" "RP2040")
     (attr through_hole)
-    (fp_text reference "J3" (at 0 -2.33) (layer "F.SilkS")
+    (fp_text reference "J3" (at 0 -2.33) (layer "F.SilkS") hide
       (effects (font (size 1 1) (thickness 0.15)))
     )
@@
     (property "Sheetname" "FootSwitches")
     (attr through_hole)
-    (fp_text reference "J8" (at 0 -2.33 90) (layer "F.SilkS")
+    (fp_text reference "J8" (at 0 -2.33 90) (layer "F.SilkS") hide
       (effects (font (size 1 1) (thickness 0.15)))
     )
@@
   (gr_arc (start 114.105 115.5) (end 110.105 115.5) (angle -90) (layer "Edge.Cuts") (width 0.1))
   (gr_line (start 182.605 119.5) (end 114.105 119.5) (layer "Edge.Cuts") (width 0.1))
+  (gr_text "~RST" (at 181.95 87.45) (layer "F.SilkS")
+    (effects (font (size 1 1) (thickness 0.15)))
+  )
+  (gr_text "GND" (at 166.05 73.35 90) (layer "F.SilkS")
+    (effects (font (size 1 0.8) (thickness 0.15)))
+  )
+  (gr_text "GND" (at 181.55 97.55) (layer "F.SilkS")
+    (effects (font (size 1 1) (thickness 0.15)))
+  )
+  (gr_text "CLK" (at 181.45 94.95) (layer "F.SilkS")
+    (effects (font (size 1 1) (thickness 0.15)))
+  )
+  (gr_text "Foot Switch\n3" (at 157.25 117.5) (layer "F.SilkS")
+    (effects (font (size 1 1) (thickness 0.15)))
+  )
+  (gr_text "3v3" (at 173.65 73.4 90) (layer "F.SilkS")
+    (effects (font (size 1 0.8) (thickness 0.15)))
+  )
+  (gr_text "MiDi" (at 176.2 75.85 90) (layer "F.SilkS")
+    (effects (font (size 1 1) (thickness 0.15)))
+  )
+  (gr_text "Foot Switch\n4" (at 172.45 117.5) (layer "F.SilkS")
+    (effects (font (size 1 1) (thickness 0.15)))
+  )
+  (gr_text "Foot Switch\n1" (at 125.8 117.45) (layer "F.SilkS")
+    (effects (font (size 1 1) (thickness 0.15)))
+  )
+  (gr_text "SWD" (at 181.6 100.1) (layer "F.SilkS")
+    (effects (font (size 1 1) (thickness 0.15)))
+  )
+  (gr_text "GND" (at 158.35 73.3 90) (layer "F.SilkS")
+    (effects (font (size 1 0.8) (thickness 0.15)))
+  )
+  (gr_text "GND" (at 181.9 84.8) (layer "F.SilkS")
+    (effects (font (size 1 1) (thickness 0.15)))
+  )
+  (gr_text "OUT" (at 171.15 73.45 90) (layer "F.SilkS")
+    (effects (font (size 1 0.8) (thickness 0.15)))
+  )
+  (gr_text "Foot Switch\n2" (at 141.25 117.5) (layer "F.SilkS")
+    (effects (font (size 1 1) (thickness 0.15)))
+  )
+  (gr_text "GND" (at 168.6 73.35 90) (layer "F.SilkS")
+    (effects (font (size 1 0.8) (thickness 0.15)))
+  )
+  (gr_text "BOOT\n" (at 155.85 73.3 90) (layer "F.SilkS")
+    (effects (font (size 1 0.7) (thickness 0.15)))
+  )
   (segment (start 160.7 94.65) (end 159.75 95.6) (width 0.16) (layer "F.Cu") (net 1))
   (segment (start 159.75 99.605) (end 159.355 100) (width 0.16) (layer "F.Cu") (net 1))
