File: stomp_control/usb.kicad_sch (KiCad schematic)
At the start: 3 parts

Commit message: initial board layout
Parts:
- J?1: renamed from J??; footprint (none) -> USB4085-GF-A:GCT_USB4085-GF-A_REVA
- R10, R9: renamed from R?; footprint (none) -> Resistor_SMD:R_0603_1608Metric_Pad0.98x0.95mm_HandSolder
Changed lines of the file:
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@@
     (stroke (width 0) (type solid) (color 0 0 0 0))
+  )
+  (label "USB_+" (at 172.72 76.2 180)
+    (effects (font (size 1.27 1.27)) (justify right bottom))
+  )
+  (label "USB_-" (at 172.72 83.82 180)
+    (effects (font (size 1.27 1.27)) (justify right bottom))
   )
   (hierarchical_label "VBUS" (shape input) (at 180.34 71.12 0)
@@
   (symbol (lib_id "power:GND") (at 107.95 121.92 0) (unit 1)
     (in_bom yes) (on_board yes)
-    (property "Reference" "#PWR?" (id 0) (at 107.95 128.27 0)
+    (property "Reference" "#PWR0122" (id 0) (at 107.95 128.27 0)
       (effects (font (size 1.27 1.27)) hide)
     )
@@
   (symbol (lib_id "power:GND") (at 149.86 121.92 0) (unit 1)
     (in_bom yes) (on_board yes)
-    (property "Reference" "#PWR?" (id 0) (at 149.86 128.27 0)
+    (property "Reference" "#PWR0121" (id 0) (at 149.86 128.27 0)
       (effects (font (size 1.27 1.27)) hide)
     )
@@
   (symbol (lib_id "Device:R_Small_US") (at 149.86 100.33 0) (unit 1)
     (in_bom yes) (on_board yes)
-    (property "Reference" "R?" (id 0) (at 147.32 99.06 0)
+    (property "Reference" "R9" (id 0) (at 147.32 99.06 0)
       (effects (font (size 1.27 1.27)) (justify right))
     )
@@
       (effects (font (size 1.27 1.27)) (justify right))
     )
-    (property "Footprint" "" (id 2) (at 149.86 100.33 0)
+    (property "Footprint" "Resistor_SMD:R_0603_1608Metric_Pad0.98x0.95mm_HandSolder" (id 2) (at 149.86 100.33 0)
       (effects (font (size 1.27 1.27)) hide)
     )
@@
   (symbol (lib_id "Device:R_Small_US") (at 154.94 100.33 0) (unit 1)
     (in_bom yes) (on_board yes)
-    (property "Reference" "R?" (id 0) (at 157.48 99.06 0)
+    (property "Reference" "R10" (id 0) (at 157.48 99.06 0)
       (effects (font (size 1.27 1.27)) (justify left))
     )
@@
       (effects (font (size 1.27 1.27)) (justify left))
     )
-    (property "Footprint" "" (id 2) (at 154.94 100.33 0)
+    (property "Footprint" "Resistor_SMD:R_0603_1608Metric_Pad0.98x0.95mm_HandSolder" (id 2) (at 154.94 100.33 0)
       (effects (font (size 1.27 1.27)) hide)
     )
@@
   (symbol (lib_id "usb_c_receptacle_usb2.0:USB_C_Receptacle_USB2.0") (at 115.57 86.36 0) (unit 1)
     (in_bom yes) (on_board yes)
-    (property "Reference" "J??" (id 0) (at 119.38 63.5 0))
+    (property "Reference" "J?1" (id 0) (at 119.38 63.5 0))
     (property "Value" "USB_C_Receptacle_USB2.0" (id 1) (at 119.38 66.04 0))
-    (property "Footprint" "" (id 2) (at 119.38 86.36 0)
+    (property "Footprint" "USB4085-GF-A:GCT_USB4085-GF-A_REVA" (id 2) (at 119.38 86.36 0)
       (effects (font (size 1.27 1.27)) hide)
     )
