File: stomp_control/cpu.kicad_sch (KiCad schematic)
At the start: 18 parts

Commit message: initial board layout
Parts:
- removed Y?: 12MHz, symbol Device:Crystal_GND2
- added Y1: 12MHz, sc_custom:ABLS-12.000MHZ-20-B-3-H-T, symbol Device:Crystal
- C1, C2: renamed from C?; value 100n -> 15p; footprint (none) -> Capacitor_SMD:C_0603_1608Metric_Pad1.08x0.95mm_HandSolder
- C3, C4, C5, C6: renamed from C?; footprint (none) -> Capacitor_SMD:C_0603_1608Metric_Pad1.08x0.95mm_HandSolder
- J1: renamed from J?; footprint (none) -> Connector_PinHeader_2.54mm:PinHeader_1x03_P2.54mm_Vertical
- J2, J3: renamed from J?; footprint (none) -> Connector_PinHeader_2.54mm:PinHeader_1x02_P2.54mm_Vertical
- R1, R2, R3, R4, R5, R6: renamed from R?; footprint (none) -> Resistor_SMD:R_0603_1608Metric_Pad0.98x0.95mm_HandSolder
- U2: renamed from U?; footprint QFN40P700X700X90-57N -> Package_DFN_QFN:QFN-56-1EP_7x7mm_P0.4mm_EP5.6x5.6mm
- gave numbers to parts that had none: 1
Connections:
- net at C1.2, R1.1, U2.20 (XIN): now also Y1.1
- net at C2.1, R3.2: now also Y1.2
- net RP_USB_-: now reaches R6.1, U2.47 (USB_DP)
- net RP_USB_+: now reaches R5.1, U2.46 (USB_DM)
Other:
- moved on the sheet: C1, C2, R3, R5, R6

Commit message: add silkscreen annotations
Parts:
- removed J2: PROG_MODE, Connector_PinHeader_2.54mm:PinHeader_1x02_P2.54mm_Vertical, symbol Connector:Conn_01x02_Female
Changed lines of the file:
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@@
-    (pin "2")
-  )
-  (symbol (lib_id "Connector:Conn_01x02_Female") (at 43.18 161.29 0) (mirror y) (unit 1)
-    (in_bom yes) (on_board yes)
-    (property "Reference" "J2" (id 0) (at 39.37 161.29 0)
-      (effects (font (size 1.27 1.27)) (justify right))
-    )
-    (property "Value" "PROG_MODE" (id 1) (at 30.48 163.83 0)
-      (effects (font (size 1.27 1.27)) (justify right))
-    )
-    (property "Footprint" "Connector_PinHeader_2.54mm:PinHeader_1x02_P2.54mm_Vertical" (id 2) (at 43.18 161.29 0)
-      (effects (font (size 1.27 1.27)) hide)
-    )
-    (property "Datasheet" "~" (id 3) (at 43.18 161.29 0)
-      (effects (font (size 1.27 1.27)) hide)
-    )
-    (pin "1")
     (pin "2")
   )
